File: g2_motor_shield.kicad_pcb (KiCad board)
At the start: 2 copper layers, 114.3 x 85.3 mm, 11 parts, among them J1 Spindle, J2 Cooling, J3 X limits, J4 Y limits, J5 Z limits, J6 Buttons, J7 Interlock, M1 TB67S249FTG, M2 TB67S249FTG, M3 TB67S249FTG

Commit message: toward a prototype
Parts:
- added REF**: MountingHole_3mm_Pad, MountingHole:MountingHole_3mm_Pad, F.Cu at (-245.1, -502.7)
- added REF**: MountingHole_3mm_Pad, MountingHole:MountingHole_3mm_Pad, F.Cu at (-245.1, -575.1)
- added REF**: MountingHole_3mm_Pad, MountingHole:MountingHole_3mm_Pad, F.Cu at (-143.5, -575.1)
- added REF**: MountingHole_3mm_Pad, MountingHole:MountingHole_3mm_Pad, F.Cu at (-143.5, -502.7)
Other:
- board size 114.3 x 85.3 mm -> 114.3 x 85.1 mm
Changed lines of the file:
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@@
   (general
     (thickness 1.6)
-    (drawings 4)
+    (drawings 6)
     (tracks 294)
     (zones 0)
-    (modules 11)
+    (modules 15)
     (nets 128)
   )
@@
     (pad_to_mask_clearance 0.051)
     (solder_mask_min_width 0.25)
-    (aux_axis_origin 0 0)
+    (aux_axis_origin -251.46 -496.316)
+    (grid_origin -251.46 -496.316)
     (visible_elements FFFFFF7F)
     (pcbplotparams
-      (layerselection 0x010fc_ffffffff)
+      (layerselection 0x01000_ffffffff)
       (usegerberextensions false)
       (usegerberattributes false)
@@
       (outputformat 1)
       (mirror false)
-      (drillshape 1)
+      (drillshape 0)
       (scaleselection 1)
-      (outputdirectory ""))
+      (outputdirectory "output/"))
   )
   (net 0 "")
@@
     )
   )
+  (module MountingHole:MountingHole_3mm_Pad (layer F.Cu)
+    (at -245.11 -502.666)
+    (descr "Mounting Hole 3mm")
+    (tags "mounting hole 3mm")
+    (attr virtual)
+    (fp_text reference REF** (at 0 -4) (layer F.SilkS)
+      (effects (font (size 1 1) (thickness 0.15)))
+    )
+    (fp_text value MountingHole_3mm_Pad (at 0 4) (layer F.Fab)
+      (effects (font (size 1 1) (thickness 0.15)))
+    )
+    (fp_circle (center 0 0) (end 3.25 0) (layer F.CrtYd) (width 0.05))
+    (fp_circle (center 0 0) (end 3 0) (layer Cmts.User) (width 0.15))
+    (fp_text user %R (at 0.3 0) (layer F.Fab)
+      (effects (font (size 1 1) (thickness 0.15)))
+    )
+    (pad 1 thru_hole circle (at 0 0) (size 6 6) (drill 3) (layers *.Cu *.Mask))
+  )
+  (module MountingHole:MountingHole_3mm_Pad (layer F.Cu)
+    (at -245.11 -575.056)
+    (descr "Mounting Hole 3mm")
+    (tags "mounting hole 3mm")
+    (attr virtual)
+    (fp_text reference REF** (at 0 -4) (layer F.SilkS)
+      (effects (font (size 1 1) (thickness 0.15)))
+    )
+    (fp_text value MountingHole_3mm_Pad (at 0 4) (layer F.Fab)
+      (effects (font (size 1 1) (thickness 0.15)))
+    )
+    (fp_circle (center 0 0) (end 3.25 0) (layer F.CrtYd) (width 0.05))
+    (fp_circle (center 0 0) (end 3 0) (layer Cmts.User) (width 0.15))
+    (fp_text user %R (at 0.3 0) (layer F.Fab)
+      (effects (font (size 1 1) (thickness 0.15)))
+    )
+    (pad 1 thru_hole circle (at 0 0) (size 6 6) (drill 3) (layers *.Cu *.Mask))
+  )
+  (module MountingHole:MountingHole_3mm_Pad (layer F.Cu)
+    (at -143.51 -575.056)
+    (descr "Mounting Hole 3mm")
+    (tags "mounting hole 3mm")
+    (attr virtual)
+    (fp_text reference REF** (at 0 -4) (layer F.SilkS)
+      (effects (font (size 1 1) (thickness 0.15)))
+    )
+    (fp_text value MountingHole_3mm_Pad (at 0 4) (layer F.Fab)
+      (effects (font (size 1 1) (thickness 0.15)))
+    )
+    (fp_circle (center 0 0) (end 3.25 0) (layer F.CrtYd) (width 0.05))
+    (fp_circle (center 0 0) (end 3 0) (layer Cmts.User) (width 0.15))
+    (fp_text user %R (at 0.3 0) (layer F.Fab)
+      (effects (font (size 1 1) (thickness 0.15)))
+    )
+    (pad 1 thru_hole circle (at 0 0) (size 6 6) (drill 3) (layers *.Cu *.Mask))
+  )
+  (module MountingHole:MountingHole_3mm_Pad (layer F.Cu)
+    (at -143.51 -502.666)
+    (descr "Mounting Hole 3mm")
+    (tags "mounting hole 3mm")
+    (attr virtual)
+    (fp_text reference REF** (at 0 -4) (layer F.SilkS)
+      (effects (font (size 1 1) (thickness 0.15)))
+    )
+    (fp_text value MountingHole_3mm_Pad (at 0 4) (layer F.Fab)
+      (effects (font (size 1 1) (thickness 0.15)))
+    )
+    (fp_circle (center 0 0) (end 3.25 0) (layer F.CrtYd) (width 0.05))
+    (fp_circle (center 0 0) (end 3 0) (layer Cmts.User) (width 0.15))
+    (fp_text user %R (at 0.3 0) (layer F.Fab)
+      (effects (font (size 1 1) (thickness 0.15)))
+    )
+    (pad 1 thru_hole circle (at 0 0) (size 6 6) (drill 3) (layers *.Cu *.Mask))
+  )
+  (dimension 72.39 (width 0.3) (layer F.SilkS)
+    (gr_text "72.390 mm" (at -129.98 -538.861 270) (layer F.SilkS)
+      (effects (font (size 1.5 1.5) (thickness 0.3)))
+    )
+    (feature1 (pts (xy -143.51 -502.666) (xy -131.493579 -502.666)))
+    (feature2 (pts (xy -143.51 -575.056) (xy -131.493579 -575.056)))
+    (crossbar (pts (xy -132.08 -575.056) (xy -132.08 -502.666)))
+    (arrow1a (pts (xy -132.08 -502.666) (xy -132.666421 -503.792504)))
+    (arrow1b (pts (xy -132.08 -502.666) (xy -131.493579 -503.792504)))
+    (arrow2a (pts (xy -132.08 -575.056) (xy -132.666421 -573.929496)))
+    (arrow2b (pts (xy -132.08 -575.056) (xy -131.493579 -573.929496)))
+  )
+  (dimension 101.6 (width 0.3) (layer F.SilkS)
+    (gr_text "101.600 mm" (at -194.31 -587.315999) (layer F.SilkS)
+      (effects (font (size 1.5 1.5) (thickness 0.3)))
+    )
+    (feature1 (pts (xy -245.11 -575.056) (xy -245.11 -585.80242)))
+    (feature2 (pts (xy -143.51 -575.056) (xy -143.51 -585.80242)))
+    (crossbar (pts (xy -143.51 -585.215999) (xy -245.11 -585.215999)))
+    (arrow1a (pts (xy -245.11 -585.215999) (xy -243.983496 -585.80242)))
+    (arrow1b (pts (xy -245.11 -585.215999) (xy -243.983496 -584.629578)))
+    (arrow2a (pts (xy -143.51 -585.215999) (xy -144.636504 -585.80242)))
+    (arrow2b (pts (xy -143.51 -585.215999) (xy -144.636504 -584.629578)))
+  )
   (gr_line (start -137.16 -496.316) (end -251.46 -496.316) (layer Edge.Cuts) (width 0.15))
-  (gr_line (start -137.16 -581.66) (end -137.16 -496.316) (layer Edge.Cuts) (width 0.15))
-  (gr_line (start -251.46 -581.66) (end -137.16 -581.66) (layer Edge.Cuts) (width 0.15))
-  (gr_line (start -251.46 -496.316) (end -251.46 -581.66) (layer Edge.Cuts) (width 0.15))
+  (gr_line (start -137.16 -581.406) (end -137.16 -496.316) (layer Edge.Cuts) (width 0.15))
+  (gr_line (start -251.46 -581.406) (end -137.16 -581.406) (layer Edge.Cuts) (width 0.15))
+  (gr_line (start -251.46 -496.316) (end -251.46 -581.406) (layer Edge.Cuts) (width 0.15))
   (segment (start -180.34 -574.77) (end -180.34 -572.77) (width 0.8) (layer B.Cu) (net 1))
   (segment (start -179.939999 -575.170001) (end -180.34 -574.77) (width 0.8) (layer B.Cu) (net 1))
